Commit message: for naming convention

File: ur5e/ros2srrc_ur5e_gazebo/urdf/ur5.urdf.xacro (robot description, xacro)
@@ -56,5 +56,5 @@
 <robot xmlns:xacro="http://wiki.ros.org/xacro" name="ur5">
   <!-- Load and initialise UR5 INITIAL POSITIONS FILE:
-  <xacro:arg name="initial_positions_file" default="$(find ur5_ros2_gazebo/config/initial_positions.yaml"/>
+  <xacro:arg name="initial_positions_file" default="$(find ros2srrc_ur5e_gazebo/config/initial_positions.yaml"/>
   <xacro:property name="initial_positions_file" default="$(arg initial_positions_file)"/> -->
   <!-- IF ADD TO UR5: initial_positions="${load_yaml(initial_positions_file)}" -->
@@ -73,5 +73,5 @@
   <xacro:arg name="safety_k_position" default="20"/>
   <!-- Include XACRO-MACRO file of the UR5 ROBOT: -->
-  <xacro:include filename="$(find ur5_ros2_gazebo)/urdf/ur5_macro.urdf.xacro"/>
+  <xacro:include filename="$(find ros2srrc_ur5e_gazebo)/urdf/ur5_macro.urdf.xacro"/>
   <xacro:ur5
     prefix=""

File: ur5e/ros2srrc_ur5e_gazebo/urdf/ur5_common.xacro (robot description, xacro)
@@ -66,5 +66,5 @@
   <xacro:macro name="ur5_common">
     <!-- ***** PARAMETER VALUES ***** -->
-    <!-- All parameter values have been taken from the following .yaml files, located in the ~/ur5_ros2_gazebo/config folder:
+    <!-- All parameter values have been taken from the following .yaml files, located in the ~/ros2srrc_ur5e_gazebo/config folder:
           - default_kinematics.yaml
           - joint_limits.yaml

File: ur5e/ros2srrc_ur5e_gazebo/urdf/ur5_macro.urdf.xacro (robot description, xacro)
@@ -58,10 +58,10 @@
   <xacro:macro name="ur5" params="prefix EE_no safety_limits safety_pos_margin safety_k_position">
     <!-- Load UR5 ROBOT TRANSMISSION file: -->
-    <xacro:include filename="$(find ur5_ros2_gazebo)/urdf/ur5_transmission.xacro" />
+    <xacro:include filename="$(find ros2srrc_ur5e_gazebo)/urdf/ur5_transmission.xacro" />
     <xacro:ur5_transmission
       prefix=""
     />
     <!-- Load UR5 ROBOT ROS2_CONTROL file: -->
-    <xacro:include filename="$(find ur5_ros2_gazebo)/urdf/ur5_ros2control.xacro" />
+    <xacro:include filename="$(find ros2srrc_ur5e_gazebo)/urdf/ur5_ros2control.xacro" />
     <xacro:ur5_ros2control
       prefix=""
@@ -69,5 +69,5 @@
     />
     <!-- Load UR5 SPECIFICATIONS file: -->
-    <xacro:include filename="$(find ur5_ros2_gazebo)/urdf/ur5_common.xacro" />
+    <xacro:include filename="$(find ros2srrc_ur5e_gazebo)/urdf/ur5_common.xacro" />
     <xacro:ur5_common/>
     <!-- ***** ur5 ROBOT .urdf SERIAL CHAIN *****-->
@@ -78,5 +78,5 @@
         <origin xyz="0 0 0" rpy="0 0 ${pi}"/>
         <geometry>
-          <mesh filename="file://$(find ur5_ros2_gazebo)/meshes/visual/base.dae"/>
+          <mesh filename="file://$(find ros2srrc_ur5e_gazebo)/meshes/visual/base.dae"/>
         </geometry>
         <material name="LightGrey">
@@ -87,5 +87,5 @@
         <origin xyz="0 0 0" rpy="0 0 ${pi}"/>
         <geometry>
-          <mesh filename="file://$(find ur5_ros2_gazebo)/meshes/collision/base.stl"/>
+          <mesh filename="file://$(find ros2srrc_ur5e_gazebo)/meshes/collision/base.stl"/>
         </geometry>
       </collision>
@@ -98,5 +98,5 @@
         <origin xyz="0 0 0" rpy="0 0 ${pi}"/>
         <geometry>
-          <mesh filename="file://$(find ur5_ros2_gazebo)/meshes/visual/shoulder.dae"/>
+          <mesh filename="file://$(find ros2srrc_ur5e_gazebo)/meshes/visual/shoulder.dae"/>
         </geometry>
         <material name="LightGrey">
@@ -107,5 +107,5 @@
         <origin xyz="0 0 0" rpy="0 0 ${pi}"/>
         <geometry>
-          <mesh filename="file://$(find ur5_ros2_gazebo)/meshes/collision/shoulder.stl"/>
+          <mesh filename="file://$(find ros2srrc_ur5e_gazebo)/meshes/collision/shoulder.stl"/>
         </geometry>
       </collision>
@@ -118,5 +118,5 @@
         <origin xyz="0 0 ${shoulder_offset}" rpy="${pi/2} 0 ${-pi/2}"/>
         <geometry>
-          <mesh filename="file://$(find ur5_ros2_gazebo)/meshes/visual/upperarm.dae"/>
+          <mesh filename="file://$(find ros2srrc_ur5e_gazebo)/meshes/visual/upperarm.dae"/>
         </geometry>
         <material name="LightGrey">
@@ -127,5 +127,5 @@
         <origin xyz="0 0 ${shoulder_offset}" rpy="${pi/2} 0 ${-pi/2}"/>
         <geometry>
-          <mesh filename="file://$(find ur5_ros2_gazebo)/meshes/collision/upperarm.stl"/>
+          <mesh filename="file://$(find ros2srrc_ur5e_gazebo)/meshes/collision/upperarm.stl"/>
         </geometry>
       </collision>
@@ -138,5 +138,5 @@
         <origin xyz="0 0 ${elbow_offset}" rpy="${pi/2} 0 ${-pi/2}"/>
         <geometry>
-          <mesh filename="file://$(find ur5_ros2_gazebo)/meshes/visual/forearm.dae"/>
+          <mesh filename="file://$(find ros2srrc_ur5e_gazebo)/meshes/visual/forearm.dae"/>
         </geometry>
         <material name="LightGrey">
@@ -147,5 +147,5 @@
         <origin xyz="0 0 ${elbow_offset}" rpy="${pi/2} 0 ${-pi/2}"/>
         <geometry>
-          <mesh filename="file://$(find ur5_ros2_gazebo)/meshes/collision/forearm.stl"/>
+          <mesh filename="file://$(find ros2srrc_ur5e_gazebo)/meshes/collision/forearm.stl"/>
         </geometry>
       </collision>
@@ -158,5 +158,5 @@
         <origin xyz="0 0 ${wrist_1_visual_offset}" rpy="${pi/2} 0 0"/>
         <geometry>
-          <mesh filename="file://$(find ur5_ros2_gazebo)/meshes/visual/wrist1.dae"/>
+          <mesh filename="file://$(find ros2srrc_ur5e_gazebo)/meshes/visual/wrist1.dae"/>
         </geometry>
         <material name="LightGrey">
@@ -167,5 +167,5 @@
         <origin xyz="0 0 ${wrist_1_visual_offset}" rpy="${pi/2} 0 0"/>
         <geometry>
-          <mesh filename="file://$(find ur5_ros2_gazebo)/meshes/collision/wrist1.stl"/>
+          <mesh filename="file://$(find ros2srrc_ur5e_gazebo)/meshes/collision/wrist1.stl"/>
         </geometry>
       </collision>
@@ -178,5 +178,5 @@
         <origin xyz="0 0 ${wrist_2_visual_offset}" rpy="0 0 0"/>
         <geometry>
-          <mesh filename="file://$(find ur5_ros2_gazebo)/meshes/visual/wrist2.dae"/>
+          <mesh filename="file://$(find ros2srrc_ur5e_gazebo)/meshes/visual/wrist2.dae"/>
         </geometry>
         <material name="LightGrey">
@@ -187,5 +187,5 @@
         <origin xyz="0 0 ${wrist_2_visual_offset}" rpy="0 0 0"/>
         <geometry>
-          <mesh filename="file://$(find ur5_ros2_gazebo)/meshes/collision/wrist2.stl"/>
+          <mesh filename="file://$(find ros2srrc_ur5e_gazebo)/meshes/collision/wrist2.stl"/>
         </geometry>
       </collision>
@@ -198,5 +198,5 @@
         <origin xyz="0 0 ${wrist_3_visual_offset}" rpy="${pi/2} 0 0"/>
         <geometry>
-          <mesh filename="file://$(find ur5_ros2_gazebo)/meshes/visual/wrist3.dae"/>
+          <mesh filename="file://$(find ros2srrc_ur5e_gazebo)/meshes/visual/wrist3.dae"/>
         </geometry>
         <material name="LightGrey">
@@ -207,5 +207,5 @@
         <origin xyz="0 0 ${wrist_3_visual_offset}" rpy="${pi/2} 0 0"/>
         <geometry>
-          <mesh filename="file://$(find ur5_ros2_gazebo)/meshes/collision/wrist3.stl"/>
+          <mesh filename="file://$(find ros2srrc_ur5e_gazebo)/meshes/collision/wrist3.stl"/>
         </geometry>
       </collision>

File: ur5e/ros2srrc_ur5e_gazebo/urdf/ur5_ros2control.xacro (robot description, xacro)
@@ -64,5 +64,5 @@
         <plugin filename="libgazebo_ros2_control.so" name="gazebo_ros2_control">
           <robot_sim_type>gazebo_ros2_control/GazeboSystem</robot_sim_type>
-          <parameters>$(find ur5_ros2_gazebo)/config/ur5_controller.yaml</parameters>
+          <parameters>$(find ros2srrc_ur5e_gazebo)/config/ur_controller.yaml</parameters>
         </plugin>
       </gazebo>
