Commit message: for ur5e

File: ur5e/ros2srrc_ur5e_gazebo/urdf/ur5e.urdf.xacro (robot description, xacro)
@@ -26,5 +26,5 @@
 # ===================================== COPYRIGHT ===================================== #
 #                                                                                       #
-#  Some of the information used to build the ROS2 UR5-Robot .urdf files in this ROS2    #
+#  Some of the information used to build the ROS2 UR5e-Robot .urdf files in this ROS2    #
 #  repository has been taken from the following resources:                              #
 #       - Universal Robots ROS2 Description:                                            #
@@ -54,9 +54,9 @@
 # IFRA (2022) ROS2.0 ROBOT SIMULATION. URL: https://github.com/IFRA-Cranfield/ros2_RobotSimulation.
 -->
-<robot xmlns:xacro="http://wiki.ros.org/xacro" name="ur5">
-  <!-- Load and initialise UR5 INITIAL POSITIONS FILE:
+<robot xmlns:xacro="http://wiki.ros.org/xacro" name="ur5e">
+  <!-- Load and initialise UR5e INITIAL POSITIONS FILE:
   <xacro:arg name="initial_positions_file" default="$(find ros2srrc_ur5e_gazebo/config/initial_positions.yaml"/>
   <xacro:property name="initial_positions_file" default="$(arg initial_positions_file)"/> -->
-  <!-- IF ADD TO UR5: initial_positions="${load_yaml(initial_positions_file)}" -->
+  <!-- IF ADD TO UR5e: initial_positions="${load_yaml(initial_positions_file)}" -->
   <!-- ===== ARGUMENTS ===== -->
   <!-- CELL LAYOUT:  -->
@@ -72,7 +72,7 @@
   <xacro:arg name="safety_pos_margin" default="0.15"/>
   <xacro:arg name="safety_k_position" default="20"/>
-  <!-- Include XACRO-MACRO file of the UR5 ROBOT: -->
-  <xacro:include filename="$(find ros2srrc_ur5e_gazebo)/urdf/ur5_macro.urdf.xacro"/>
-  <xacro:ur5
+  <!-- Include XACRO-MACRO file of the UR5e ROBOT-->
+  <xacro:include filename="$(find ros2srrc_ur5e_gazebo)/urdf/ur5e_macro.urdf.xacro"/>
+  <xacro:ur5e
     prefix=""
     EE_no="${EE_no}"

File: ur5e/ros2srrc_ur5e_gazebo/urdf/ur5e_macro.urdf.xacro (robot description, xacro)
@@ -24,7 +24,6 @@
 #                                                                                       #
 # ===================================== COPYRIGHT ===================================== #
-# ===================================== COPYRIGHT ===================================== #
-#                                                                                       #
-#  Some of the information used to build the ROS2 UR5-Robot .urdf files in this ROS2    #
+[ERROR] [launch]: Caught exception in launch (see debug for traceback): Caught exception when trying to load file of format [py]: not well-formed (invalid token): line 216, column 19
+Some of the information used to build the ROS2 UR5-Robot .urdf files in this ROS2    #
 #  repository has been taken from the following resources:                              #
 #       - Universal Robots ROS2 Description:                                            #
@@ -36,8 +35,6 @@
 #       - ROS-Industrial - https://rosindustrial.org                                    #
 #       - Universal Robots - https://github.com/UniversalRobots                         #
-#       - Nadia Hammoudeh Garcia, Kelsey Hawkins, G.A. vd. Hoorn, Lovro Ivanov, Mathias #
-#         Ludtke, Wim Meeussen, Felix Messmer, Miguel Prada Sarasola, Denis Stogl,      #
-#         Andy Zelenak, Marvin Grosse Besselmann.                                       #
-#       - Maintainers: Felix Exner (exner@fzi.de), Tristan Schnell (schnell@fzi.de),    #
+#  [ERROR] [launch]: Caught exception in launch (see debug for traceback): Caught exception when trying to load file of format [py]: not well-formed (invalid token): line 216, column 19
+     - Maintainers: Felix Exner (exner@fzi.de), Tristan Schnell (schnell@fzi.de),    #
 #         Lovro Ivanov (lovro.ivanov@gmail.com), Denis Stogl (denis@stoglrobotics.de).  #
 #                                                                                       #
@@ -55,21 +52,21 @@
 -->
 <robot xmlns:xacro="http://wiki.ros.org/xacro">
-  <!-- XACRO-MACRO of UR5 ROBOT: -->
-  <xacro:macro name="ur5" params="prefix EE_no safety_limits safety_pos_margin safety_k_position">
-    <!-- Load UR5 ROBOT TRANSMISSION file: -->
-    <xacro:include filename="$(find ros2srrc_ur5e_gazebo)/urdf/ur5_transmission.xacro" />
-    <xacro:ur5_transmission
+  <!-- XACRO-MACRO of UR5e ROBOT: -->
+  <xacro:macro name="ur5e" params="prefix EE_no safety_limits safety_pos_margin safety_k_position">
+    <!-- Load UR5e ROBOT TRANSMISSION file: -->
+    <xacro:include filename="$(find ros2srrc_ur5e_gazebo)/urdf/ur5e_transmission.xacro" />
+    <xacro:ur5e_transmission
       prefix=""
     />
-    <!-- Load UR5 ROBOT ROS2_CONTROL file: -->
-    <xacro:include filename="$(find ros2srrc_ur5e_gazebo)/urdf/ur5_ros2control.xacro" />
+    <!-- Load UR5e ROBOT ROS2_CONTROL file: -->
+    <xacro:include filename="$(find ros2srrc_ur5e_gazebo)/urdf/ur5e_ros2control.xacro" />
     <xacro:ur5_ros2control
       prefix=""
       EE_no="${EE_no}"
     />
-    <!-- Load UR5 SPECIFICATIONS file: -->
-    <xacro:include filename="$(find ros2srrc_ur5e_gazebo)/urdf/ur5_common.xacro" />
+    <!-- Load UR5e SPECIFICATIONS file: -->
+    <xacro:include filename="$(find ros2srrc_ur5e_gazebo)/urdf/ur5e_common.xacro" />
     <xacro:ur5_common/>
-    <!-- ***** ur5 ROBOT .urdf SERIAL CHAIN *****-->
+    <!-- ***** ur5e ROBOT .urdf SERIAL CHAIN *****-->
     <!-- Links: -->
     <link name="${prefix}base_link"/>
@@ -80,5 +77,5 @@
           <mesh filename="file://$(find ros2srrc_ur5e_gazebo)/meshes/visual/base.dae"/>
         </geometry>
-        <material name="LightGrey">
+      <material name="LightGrey">
           <color rgba="0.7 0.7 0.7 1.0"/>
         </material>
@@ -123,5 +120,5 @@
           <color rgba="0.7 0.7 0.7 1.0"/>
         </material>
-      </visual>
+   </visual>
       <collision>
         <origin xyz="0 0 ${shoulder_offset}" rpy="${pi/2} 0 ${-pi/2}"/>
@@ -131,8 +128,8 @@
       </collision>
       <xacro:cylinder_inertial radius="${upperarm_inertia_radius}" length="${upperarm_inertia_length}" mass="${upper_arm_mass}">
-        <origin xyz="${-0.5 * upperarm_inertia_length} 0.0 ${upper_arm_inertia_offset}" rpy="0 ${pi/2} 0" />
-      </xacro:cylinder_inertial>
-    </link>
-    <link name="${prefix}forearm_link">
+         <origin xyz="${-0.5 * upperarm_inertia_length} 0.0 ${upper_arm_inertia_offset}" rpy="0 ${pi/2} 0" />
+      </xacro:cylinder_inertial>
+    </link>
+  <link name="${prefix}forearm_link">
       <visual>
         <origin xyz="0 0 ${elbow_offset}" rpy="${pi/2} 0 ${-pi/2}"/>
@@ -146,5 +143,5 @@
       <collision>
         <origin xyz="0 0 ${elbow_offset}" rpy="${pi/2} 0 ${-pi/2}"/>
-        <geometry>
+     <geometry>
           <mesh filename="file://$(find ros2srrc_ur5e_gazebo)/meshes/collision/forearm.stl"/>
         </geometry>
@@ -161,5 +158,5 @@
         </geometry>
         <material name="LightGrey">
-          <color rgba="0.7 0.7 0.7 1.0"/>
+      <color rgba="0.7 0.7 0.7 1.0"/>
         </material>
       </visual>

File: ur5e/ros2srrc_ur5e_gazebo/urdf/ur5e_transmission.xacro (robot description, xacro)
@@ -47,5 +47,6 @@
 #  CHANGES MADE:                                                                        #
 #  Robot information/specifications have been taken, and the code has been modified and #
-#  re-organised in accordance with the ros2_RobotSimulation standards.                  #
+#  re-or[ERROR] [launch]: Caught exception in launch (see debug for traceback): Caught exception when trying to load file of format [py]: not well-formed (invalid token): line 216, column 19
+ganised in accordance with the ros2_RobotSimulation standards.                  #
 #                                                                                       #
 # ===================================== COPYRIGHT ===================================== #
@@ -55,5 +56,5 @@
 -->
 <robot xmlns:xacro="http://wiki.ros.org/xacro">
-  <xacro:macro name="ur5_transmission" params="prefix">
+  <xacro:macro name="ur5e_transmission" params="prefix">
     <transmission name="${prefix}shoulder_pan_trans">
       <type>transmission_interface/SimpleTransmission</type>
